File: Schematic/Main.brd (EAGLE design)
At the start: 160 x 100 mm, 83 parts, among them IC1 PIC18F4550_40, IC2 7805, IC3 ACS714, IC4 AD7734, IC5 AD780, IC6 AD5292, IC8 ACS714, IC9 AD5292, K1 SRD-24VDC-SL-C, K2 SRD-24VDC-SL-C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

Commit message: Swapped PIC for AVR.
Parts:
- removed PL1: ICSP, jason-test:6X1-ICSP
- removed Q1: 20MHz, crystal:HC49/S
- removed R10: 470R, rcl:R2012
- removed R9: 10k, rcl:R2012
- removed X1: USBPTH, SparkFun:USB-B-PTH
- added C1: 0.1uF, rcl:C2012
- added C24, C33: 10uF, rcl:E2,5-5
- added IC7: MAX232, maxim:DIL16
- added Q3: 20MHz, crystal:HC49/S
- added SV10: (no value), con-lstb:MA03-1
- added SV7: (no value), con-lstb:MA05-2
- added SV8: (no value), con-lstb:MA10-1
- added SV9: (no value), con-lstb:MA03-2
- C16: value 0.1uF -> 10uF; device rcl:C025-030X050 -> rcl:E2,5-5
- C2, C3: value 0.1uF -> 22pF; device rcl:C2012 -> rcl:C025-024X044
- C4: value 0.1uF -> 10uF; device rcl:C2012 -> rcl:E2,5-5
- IC1: value PIC18F4550_40 -> ATMEGA644-20PU; device microchip:DIL40 -> atmel:DIL40
- moved C16 316.8 mm to (-101.6, -227.3)
- moved C4 315.2 mm to (-101.6, -221.0)
- moved C3 241.3 mm to (-101.6, -167.6)
- moved C2 236.4 mm to (-101.6, -162.6)
- moved IC1 171.4 mm to (-74.9, -134.6)
Connections:
- new net MISO: IC1.7, SV7.9
- new net MOSI: IC1.6, SV7.1
- new net N$28: IC1.24, SV8.6
- new net N$34: IC1.22, SV8.8
- new net N$35: IC7.13, SV9.5
- new net N$36: IC7.14, SV9.4
- new net N$37: C24.-, IC7.5
- new net N$38: C16.-, IC7.3
- new net N$45: C24.+, IC7.4
- new net N$48: C16.+, IC7.1
- new net N$49: C33.-, IC7.6
- new net N$50: C4.+, IC7.2
- new net RS232_RX: SV10.1, SV9.6
- new net RS232_TX: SV10.2, SV9.3
- new net SCK: IC1.8, SV7.7
- new net UART_RX: IC1.14, IC7.12
- new net UART_TX: IC1.15, IC7.11
- new net VCC: IC7.16
- net !ADC_CS!: now also IC1.3; no longer IC1.27
- net !CH1_CS!: now also IC1.4; no longer IC1.28
- net !CH2_CS!: now also IC1.5; no longer IC1.29
- net !LCD_STB!: now also IC1.38; no longer IC1.16
- net !RESET!: now also IC1.9, SV7.5; no longer IC1.1, PL1.PIN1, R10.1
- net +5V: now also C1.1, C4.-, IC1.10, IC1.30, SV7.2, SV8.9; no longer C2.1, C3.2, IC1.11, IC1.32, PL1.PIN2, R9.2
- net FAN_PWM: now also IC1.20; no longer IC1.10
- net GND: now also C1.2, C2.1, C33.+, IC1.11, IC7.15, SV10.3, SV7.10, SV7.4, SV7.6, SV7.8, SV8.10; no longer C16.1, C2.2, C4.1, IC1.12, PL1.PIN3, X1.GND
- net LCD_CLK: now also IC1.39; no longer IC1.15
- net LCD_IO: now also IC1.40; no longer IC1.7
- net N$1: now also C3.2, IC1.12, Q3.2; no longer C4.2, IC1.18
- net N$10: now also IC1.34; no longer IC1.3
- net N$11: now also IC1.33; no longer IC1.2
- net N$12: now also IC1.36; no longer IC1.5
- net N$13: now also IC1.16, R1.2; no longer IC1.13, Q1.2
- net N$14: now also IC1.29, SV8.1; no longer IC1.14, Q1.1
- net N$15: now also IC1.28, SV8.2; no longer IC1.23, X1.D-
- net N$16: now also IC1.27, SV8.3; no longer IC1.24, X1.D+
- net N$19: now also IC1.26, SV8.4; no longer IC1.21, OK2.1
- net N$2: now also C2.2, IC1.13, Q3.1; no longer C16.2, R10.2, R9.1
- net N$20: now also IC1.25, SV8.5; no longer IC1.22, OK1.1
- net N$3: now also IC1.18, OK2.1; no longer IC1.39, PL1.PIN5
- net N$30: now also IC1.23, SV8.7; no longer IC1.6, SV6.2
- net N$4: now also IC1.19, OK1.1; no longer IC1.40, PL1.PIN4
- net N$5: now also IC1.37, SV6.2; no longer IC1.19, R1.2
- net N$6: now also IC1.17; no longer IC1.20
- net N$9: now also IC1.35; no longer IC1.4
- net SPI_SCK: no longer IC1.34
- net SPI_SDI: no longer IC1.33
- net SPI_SDO: no longer IC1.26
- net SPKR: now also IC1.21; no longer IC1.36

Commit message: Connected ADC_RDY to AVR.
Connections:
- net N$10 renamed ROT_BTN
- net N$12 renamed ROT_A
- net N$9 renamed ROT_B
- net !ADC_RDY!: now also IC1.2
Changed lines of the file:
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@@
 <wire x1="-85.09" y1="96.52" x2="-69.43" y2="102.87" width="0" layer="19" extent="1-1"/>
 </signal>
-<signal name="N$9">
+<signal name="ROT_B">
 <contactref element="SV3" pad="2"/>
 <contactref element="IC1" pad="35"/>
 <wire x1="-34.29" y1="90.17" x2="-86.36" y2="-127" width="0" layer="19" extent="1-1"/>
 </signal>
-<signal name="N$10">
+<signal name="ROT_BTN">
 <contactref element="SV3" pad="3"/>
 <contactref element="IC1" pad="34"/>
@@
 <wire x1="-29.21" y1="90.17" x2="-81.28" y2="-127" width="0" layer="19" extent="1-1"/>
 </signal>
-<signal name="N$12">
+<signal name="ROT_A">
 <contactref element="SV3" pad="1"/>
 <contactref element="IC1" pad="36"/>
@@
 <signal name="!ADC_RDY!">
 <contactref element="IC4" pad="24"/>
+<contactref element="IC1" pad="2"/>
+<wire x1="-91.795" y1="85.4678" x2="-96.52" y2="-142.24" width="0" layer="19" extent="1-1"/>
 </signal>
 <signal name="N$31">

Commit message: PCB layour and stuffs.
Parts:
- removed C14, C8: 10uF, rcl:E2,5-5
- removed C18: 0.1uF, rcl:C2012
- removed C19, C21: 100pF, rcl:C2012
- removed C20, C22: 300pF, rcl:C2012
- removed D4: 1N4148, diode:DO35-7
- removed R21, R22, R23: 10k, rcl:R2012
- removed R6: 300R, rcl:R2012
- removed R7: 1k, rcl:R2012
- removed SP1: (no value), buzzer:KSS1201
- removed SV10, SV4: (no value), con-lstb:MA03-1
- added SV11: (no value), con-lstb:MA03-1
- SV9: device con-lstb:MA03-2 -> con-lstb:MA03-1
- moved C33 274.8 mm to (22.0, 5.40), turned to 90 degrees
- moved C24 266.5 mm to (16.4, 5.32)
- moved SV7 259.4 mm to (5.90, 61.2), turned to 90 degrees
- moved SV8 259.3 mm to (42.1, 36.8), turned to 270 degrees
- moved SV9 257.8 mm to (10.0, 26.0)
- moved C16 255.3 mm to (3.60, 5.33), turned to 180 degrees
- moved C4 252.1 mm to (9.02, 5.60), turned to 270 degrees
- moved C32 250.7 mm to (61.5, 69.8)
- moved C3 247.1 mm to (10.4, 52.6), turned to 315 degrees
- moved C2 238.5 mm to (7.44, 49.6), turned to 315 degrees
- moved IC7 237.0 mm to (12.6, 17.4)
- moved C1 236.4 mm to (25.5, 51.9), turned to 270 degrees
- moved Q3 230.9 mm to (13.1, 46.9), turned to 45 degrees
- moved JP4 218.1 mm to (96.4, 58.4), turned to 270 degrees
- moved C31 216.6 mm to (60.9, 29.0), turned to 180 degrees
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Connections:
- removed net 5V_2: C10.1, IC4.27
- removed net N$23: C26.2, SP1.+
- removed net N$24: R6.1, SV4.1
- removed net N$25: R7.1, SV4.2
- removed net N$35: IC7.13, SV9.5
- removed net N$36: IC7.14, SV9.4
- new net N$9: C26.2, SV11.1
- net !ADC_CS!: no longer R21.1
- net !CH1_CS!: no longer R22.1
- net !CH2_CS!: no longer R23.1
- net +5V: now also C10.1, IC4.27; no longer C18.2, R21.2, R22.2, R23.2, R6.2
- net ADC_VREF: no longer C14.+
- net AGND: no longer C20.1, C22.1
- net CH1_IOUT: no longer IC8.7
- net CH1_OUT: no longer C19.2, D4.C
- net CH1_VOUT: no longer C19.1, C20.2
- net CH2_IOUT: now also IC8.7
- net CH2_OUT: no longer C21.2
- net CH2_VOUT: no longer C21.1, C22.2
- net GND: now also SV9.2; no longer C14.-, C18.1, SV10.3, SV4.3
- net GNDI: no longer C8.-, D4.A
- net N$26: no longer C8.+
- net RS232_RX: now also IC7.13, SV9.3; no longer SV10.1, SV9.6
- net RS232_TX: now also IC7.14, SV9.1; no longer SV10.2, SV9.3
- net SPKR: now also SV11.3; no longer SP1.-
- net V+: no longer R7.2
Routing:
- net GND: track 0.00 -> 327.1 mm
- net V+: track 0.00 -> 203.9 mm, vias 0 -> 1
- net +5V: track 0.00 -> 155.0 mm, vias 0 -> 4
- net GNDI: track 0.00 -> 126.4 mm
- net AGND: track 0.00 -> 44.4 mm, vias 0 -> 2
- net CH2_IOUT: track 0.00 -> 36.8 mm
- net CH2_VOUT: track 0.00 -> 33.6 mm
- net ADC_VREF: track 0.00 -> 32.1 mm
- net CH1_VOUT: track 0.00 -> 28.9 mm, vias 0 -> 2
- net UART_RX: track 0.00 -> 28.6 mm
- net CH2_OUT: track 0.00 -> 26.0 mm
- net UART_TX: track 0.00 -> 25.8 mm
- net CH1_OUT: track 0.00 -> 24.4 mm
- net CH1_IOUT: track 0.00 -> 22.5 mm, vias 0 -> 2
- net N$22: track 0.00 -> 20.9 mm
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Other:
- board size 160 x 100 mm -> 100 x 100 mm
