File: Schematic/Main.sch (EAGLE design)
At the start: 87 parts, among them IC1 ATMEGA644-20PU, IC2 7805, IC3 ACS714, IC4 AD7734, IC5 AD780, IC6 AD5292, IC7 MAX232, IC8 ACS714, IC9 AD5292, K1 SRD-24VDC-SL-C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

Commit message: Connected ADC_RDY to AVR.
Connections:
- net N$10 renamed ROT_BTN
- net N$12 renamed ROT_A
- net N$9 renamed ROT_B
- net !ADC_RDY!: now also IC1.PCINT9/CLKO/T1_PB1
Changed lines of the file:
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@@
 <pinref part="IC1" gate="G$1" pin="AVCC"/>
 <pinref part="P+4" gate="1" pin="+5V"/>
+<junction x="30.48" y="-2.54"/>
 </segment>
 <segment>
@@
 </segment>
 </net>
-<net name="N$9" class="0">
+<net name="ROT_B" class="0">
 <segment>
 <wire x1="50.8" y1="10.16" x2="30.48" y2="10.16" width="0.1524" layer="91"/>
@@
 </segment>
 </net>
-<net name="N$10" class="0">
+<net name="ROT_BTN" class="0">
 <segment>
 <wire x1="30.48" y1="7.62" x2="50.8" y2="7.62" width="0.1524" layer="91"/>
@@
 </segment>
 </net>
-<net name="N$12" class="0">
+<net name="ROT_A" class="0">
 <segment>
 <wire x1="50.8" y1="12.7" x2="30.48" y2="12.7" width="0.1524" layer="91"/>
@@
 <label x="-101.6" y="40.64" size="1.778" layer="95" rot="R90" xref="yes"/>
 </segment>
+<segment>
+<pinref part="IC1" gate="G$1" pin="PCINT9/CLKO/T1_PB1"/>
+<wire x1="-30.48" y1="20.32" x2="-33.02" y2="20.32" width="0.1524" layer="91"/>
+<label x="-33.02" y="20.32" size="1.778" layer="95" rot="R180" xref="yes"/>
+<junction x="-30.48" y="20.32"/>
+</segment>
 </net>
 <net name="N$31" class="0">
@@
 <wire x1="30.48" y1="-5.08" x2="50.8" y2="-5.08" width="0.1524" layer="91"/>
 <junction x="50.8" y="-5.08"/>
+<junction x="30.48" y="-5.08"/>
 </segment>
 </net>
@@
 <wire x1="50.8" y1="-7.62" x2="30.48" y2="-7.62" width="0.1524" layer="91"/>
 <junction x="50.8" y="-7.62"/>
+<junction x="30.48" y="-7.62"/>
 </segment>
 </net>
@@
 <wire x1="30.48" y1="-10.16" x2="50.8" y2="-10.16" width="0.1524" layer="91"/>
 <junction x="50.8" y="-10.16"/>
+<junction x="30.48" y="-10.16"/>
 </segment>
 </net>
@@
 <wire x1="50.8" y1="-12.7" x2="30.48" y2="-12.7" width="0.1524" layer="91"/>
 <junction x="50.8" y="-12.7"/>
+<junction x="30.48" y="-12.7"/>
 </segment>
 </net>
@@
 <wire x1="30.48" y1="-15.24" x2="50.8" y2="-15.24" width="0.1524" layer="91"/>
 <junction x="50.8" y="-15.24"/>
+<junction x="30.48" y="-15.24"/>
 </segment>
 </net>
@@
 <wire x1="50.8" y1="-17.78" x2="30.48" y2="-17.78" width="0.1524" layer="91"/>
 <junction x="50.8" y="-17.78"/>
+<junction x="30.48" y="-17.78"/>
 </segment>
 </net>
@@
 <wire x1="30.48" y1="-20.32" x2="50.8" y2="-20.32" width="0.1524" layer="91"/>
 <junction x="50.8" y="-20.32"/>
+<junction x="30.48" y="-20.32"/>
 </segment>
 </net>
@@
 <wire x1="50.8" y1="-22.86" x2="30.48" y2="-22.86" width="0.1524" layer="91"/>
 <junction x="50.8" y="-22.86"/>
-</segment>
-</net>
+<junction x="30.48" y="-22.86"/>
+</segment>
+</net>

Commit message: PCB layour and stuffs.
Parts:
- removed C14, C8: 10uF, rcl:CPOL-EUE2.5-5
- removed C18: 0.1uF, rcl:C-EUC2012
- removed C19, C21: 100pF, rcl:C-EUC2012
- removed C20, C22: 300pF, rcl:C-EUC2012
- removed D4: 1N4148, diode:1N4148DO35-7
- removed R21, R22, R23: 10k, rcl:R-EU_R2012
- removed R6: 300R, rcl:R-EU_R2012
- removed R7: 1k, rcl:R-EU_R2012
- removed SP1: KSS1201, buzzer:KSS1201
- removed SV10, SV4: (no value), con-lstb:MA03-1
- added SV11: (no value), con-lstb:MA03-1
- SV9: device con-lstb:MA03-2 -> con-lstb:MA03-1; OC_FARNELL (none) -> unknown; OC_NEWARK (none) -> unknown
Connections:
- removed net 5V_2: C10.1, IC4.DVCC
- removed net N$23: C26.2, SP1.1
- removed net N$24: R6.1, SV4.1
- removed net N$25: R7.1, SV4.2
- removed net N$35: IC7G$1.R1IN, SV9.5
- removed net N$36: IC7G$1.T1OUT, SV9.4
- new net N$9: C26.2, SV11.1
- net !ADC_CS!: no longer R21.1
- net !CH1_CS!: no longer R22.1
- net !CH2_CS!: no longer R23.1
- net +5V: now also C10.1, IC4.DVCC; no longer C18.2, R21.2, R22.2, R23.2, R6.2
- net ADC_VREF: no longer C14.+
- net AGND: no longer C20.1, C22.1
- net CH1_IOUT: no longer IC8.VOUT
- net CH1_OUT: no longer C19.2, D4.C
- net CH1_VOUT: no longer C19.1, C20.2
- net CH2_IOUT: now also IC8.VOUT
- net CH2_OUT: no longer C21.2
- net CH2_VOUT: no longer C21.1, C22.2
- net GND: now also SV9.2; no longer C14.-, C18.1, SV10.3, SV4.3
- net GNDI: no longer C8.-, D4.A
- net N$26: no longer C8.+
- net RS232_RX: now also IC7G$1.R1IN, SV9.3; no longer SV10.1, SV9.6
- net RS232_TX: now also IC7G$1.T1OUT, SV9.1; no longer SV10.2, SV9.3
- net SPKR: now also SV11.3; no longer SP1.2
- net V+: no longer R7.2
Other:
- note removed: "PWRLED"
